File: SofleUnsplit.kicad_pcb (KiCad board)
At the start: 2 copper layers, 0 parts

Commit message: Left half switches
Parts:
- added D1: 1N4148W, Diode_SMD:D_SOD-123F, F.Cu at (24.3, -61.3)
- added D10: 1N4148W, Diode_SMD:D_SOD-123F, F.Cu at (24.3, -31.1)
- added D11: 1N4148W, Diode_SMD:D_SOD-123F, F.Cu at (29.8, -61.3)
- added D12: 1N4148W, Diode_SMD:D_SOD-123F, F.Cu at (29.8, -57.9)
- added D13: 1N4148W, Diode_SMD:D_SOD-123F, F.Cu at (29.8, -54.6)
- added D14: 1N4148W, Diode_SMD:D_SOD-123F, F.Cu at (29.8, -51.2)
- added D15: 1N4148W, Diode_SMD:D_SOD-123F, F.Cu at (29.8, -47.9)
- added D16: 1N4148W, Diode_SMD:D_SOD-123F, F.Cu at (29.8, -44.5)
- added D17: 1N4148W, Diode_SMD:D_SOD-123F, F.Cu at (29.8, -41.2)
- added D18: 1N4148W, Diode_SMD:D_SOD-123F, F.Cu at (29.8, -37.8)
- added D19: 1N4148W, Diode_SMD:D_SOD-123F, F.Cu at (29.8, -34.5)
- added D2: 1N4148W, Diode_SMD:D_SOD-123F, F.Cu at (24.3, -57.9)
- added D20: 1N4148W, Diode_SMD:D_SOD-123F, F.Cu at (29.8, -31.1)
- added D21: 1N4148W, Diode_SMD:D_SOD-123F, F.Cu at (35.3, -61.3)
- added D22: 1N4148W, Diode_SMD:D_SOD-123F, F.Cu at (35.3, -57.9)
- added D23: 1N4148W, Diode_SMD:D_SOD-123F, F.Cu at (35.3, -54.6)
- added D24: 1N4148W, Diode_SMD:D_SOD-123F, F.Cu at (35.3, -51.2)
- added D25: 1N4148W, Diode_SMD:D_SOD-123F, F.Cu at (35.3, -47.9)
- added D26: 1N4148W, Diode_SMD:D_SOD-123F, F.Cu at (35.3, -44.5)
- added D27: 1N4148W, Diode_SMD:D_SOD-123F, F.Cu at (35.3, -41.2)
- added D28: 1N4148W, Diode_SMD:D_SOD-123F, F.Cu at (35.3, -37.8)
- added D29: 1N4148W, Diode_SMD:D_SOD-123F, F.Cu at (35.3, -34.5)
- added D3: 1N4148W, Diode_SMD:D_SOD-123F, F.Cu at (24.3, -54.6)
- added D30: 1N4148W, Diode_SMD:D_SOD-123F, F.Cu at (35.3, -31.1)
- added D31: 1N4148W, Diode_SMD:D_SOD-123F, F.Cu at (40.8, -61.3)
- added D32: 1N4148W, Diode_SMD:D_SOD-123F, F.Cu at (40.8, -57.9)
- added D33: 1N4148W, Diode_SMD:D_SOD-123F, F.Cu at (40.8, -54.6)
- added D34: 1N4148W, Diode_SMD:D_SOD-123F, F.Cu at (40.8, -51.2)
- added D35: 1N4148W, Diode_SMD:D_SOD-123F, F.Cu at (40.8, -47.9)
- added D36: 1N4148W, Diode_SMD:D_SOD-123F, F.Cu at (40.8, -44.5)
- added D37: 1N4148W, Diode_SMD:D_SOD-123F, F.Cu at (40.8, -41.2)
- added D38: 1N4148W, Diode_SMD:D_SOD-123F, F.Cu at (40.8, -37.8)
- added D39: 1N4148W, Diode_SMD:D_SOD-123F, F.Cu at (40.8, -34.5)
- added D4: 1N4148W, Diode_SMD:D_SOD-123F, F.Cu at (24.3, -51.2)
- added D40: 1N4148W, Diode_SMD:D_SOD-123F, F.Cu at (40.8, -31.1)
- added D41: 1N4148W, Diode_SMD:D_SOD-123F, F.Cu at (46.3, -61.3)
- added D42: 1N4148W, Diode_SMD:D_SOD-123F, F.Cu at (46.3, -57.9)
- added D43: 1N4148W, Diode_SMD:D_SOD-123F, F.Cu at (46.3, -54.6)
- added D44: 1N4148W, Diode_SMD:D_SOD-123F, F.Cu at (46.3, -51.2)
- added D45: 1N4148W, Diode_SMD:D_SOD-123F, F.Cu at (46.3, -47.9)
- added D46: 1N4148W, Diode_SMD:D_SOD-123F, F.Cu at (46.3, -44.5)
- added D47: 1N4148W, Diode_SMD:D_SOD-123F, F.Cu at (46.3, -41.2)
- added D48: 1N4148W, Diode_SMD:D_SOD-123F, F.Cu at (46.3, -37.8)
- added D49: 1N4148W, Diode_SMD:D_SOD-123F, F.Cu at (46.3, -34.5)
- added D5: 1N4148W, Diode_SMD:D_SOD-123F, F.Cu at (24.3, -47.9)
- added D50: 1N4148W, Diode_SMD:D_SOD-123F, F.Cu at (46.3, -31.1)
- added D51: 1N4148W, Diode_SMD:D_SOD-123F, F.Cu at (51.8, -61.3)
- added D52: 1N4148W, Diode_SMD:D_SOD-123F, F.Cu at (51.8, -57.9)
- added D53: 1N4148W, Diode_SMD:D_SOD-123F, F.Cu at (51.8, -54.6)
- added D54: 1N4148W, Diode_SMD:D_SOD-123F, F.Cu at (51.8, -51.2)
- added D55: 1N4148W, Diode_SMD:D_SOD-123F, F.Cu at (51.8, -47.9)
- added D56: 1N4148W, Diode_SMD:D_SOD-123F, F.Cu at (51.8, -44.5)
- added D57: 1N4148W, Diode_SMD:D_SOD-123F, F.Cu at (51.8, -41.2)
- added D58: 1N4148W, Diode_SMD:D_SOD-123F, F.Cu at (51.8, -37.8)
- added D6: 1N4148W, Diode_SMD:D_SOD-123F, F.Cu at (24.3, -44.5)
- added D7: 1N4148W, Diode_SMD:D_SOD-123F, F.Cu at (24.3, -41.2)
- added D8: 1N4148W, Diode_SMD:D_SOD-123F, F.Cu at (24.3, -37.8)
- added D9: 1N4148W, Diode_SMD:D_SOD-123F, F.Cu at (24.3, -34.5)
- added SW1: Switch, zzkeeb:Switch_ChocV1-hotswap, F.Cu at (93.5, 70.0)
- added SW10: Switch, zzkeeb:Switch_ChocV1-hotswap, F.Cu at (129.5, 61.0)
- added SW11: Switch, zzkeeb:Switch_ChocV1-hotswap, F.Cu at (129.5, 78.0)
- added SW12: Switch, zzkeeb:Switch_ChocV1-hotswap, F.Cu at (129.5, 95.0)
- added SW13: Switch, zzkeeb:Switch_ChocV1-hotswap, F.Cu at (129.5, 112.0)
- added SW14: Switch, zzkeeb:Switch_ChocV1-hotswap, F.Cu at (147.5, 126.5)
- added SW15: Switch, zzkeeb:Switch_ChocV1-hotswap, F.Cu at (147.5, 58.5)
- added SW16: Switch, zzkeeb:Switch_ChocV1-hotswap, F.Cu at (147.5, 75.5)
- added SW17: Switch, zzkeeb:Switch_ChocV1-hotswap, F.Cu at (147.5, 92.5)
- added SW18: Switch, zzkeeb:Switch_ChocV1-hotswap, F.Cu at (147.5, 109.5)
- added SW19: Switch, zzkeeb:Switch_ChocV1-hotswap, F.Cu at (165.5, 129.0)
- added SW2: Switch, zzkeeb:Switch_ChocV1-hotswap, F.Cu at (93.5, 87.0)
- added SW20: Switch, zzkeeb:Switch_ChocV1-hotswap, F.Cu at (165.5, 61.0)
- added SW21: Switch, zzkeeb:Switch_ChocV1-hotswap, F.Cu at (165.5, 78.0)
- added SW22: Switch, zzkeeb:Switch_ChocV1-hotswap, F.Cu at (165.5, 95.0)
- added SW23: Switch, zzkeeb:Switch_ChocV1-hotswap, F.Cu at (165.5, 112.0)
- added SW24: Switch, zzkeeb:Switch_ChocV1-hotswap, F.Cu at (186.0, 134.6)
- added SW25: Switch, zzkeeb:Switch_ChocV1-hotswap, F.Cu at (183.5, 63.5)
- added SW26: Switch, zzkeeb:Switch_ChocV1-hotswap, F.Cu at (183.5, 80.5)
- added SW27: Switch, zzkeeb:Switch_ChocV1-hotswap, F.Cu at (183.5, 97.5)
- added SW28: Switch, zzkeeb:Switch_ChocV1-hotswap, F.Cu at (183.5, 114.5)
- added SW29: Switch, zzkeeb:Switch_ChocV1-hotswap, F.Cu at (203.6, 143.1)
- added SW3: Switch, zzkeeb:Switch_ChocV1-hotswap, F.Cu at (93.5, 104.0)
- added SW30: Switch, zzkeeb:Switch_ChocV1-hotswap, F.Cu at (258.5, 60.0)
- added SW31: Switch, zzkeeb:Switch_ChocV1-hotswap, F.Cu at (258.5, 78.2)
- added SW32: Switch, zzkeeb:Switch_ChocV1-hotswap, F.Cu at (258.5, 96.3)
- added SW33: Switch, zzkeeb:Switch_ChocV1-hotswap, F.Cu at (258.5, 114.5)
- added SW34: Switch, zzkeeb:Switch_ChocV1-hotswap, F.Cu at (235.5, 143.5)
- added SW35: Switch, zzkeeb:Switch_ChocV1-hotswap, F.Cu at (277.5, 56.5)
- added SW36: Switch, zzkeeb:Switch_ChocV1-hotswap, F.Cu at (277.5, 74.7)
- added SW37: Switch, zzkeeb:Switch_ChocV1-hotswap, F.Cu at (277.5, 96.0)
- added SW38: Switch, zzkeeb:Switch_ChocV1-hotswap, F.Cu at (277.5, 114.2)
- added SW39: Switch, zzkeeb:Switch_ChocV1-hotswap, F.Cu at (256.0, 136.0)
- added SW4: Switch, zzkeeb:Switch_ChocV1-hotswap, F.Cu at (93.5, 121.0)
- added SW40: Switch, zzkeeb:Switch_ChocV1-hotswap, F.Cu at (296.5, 54.0)
- added SW41: Switch, zzkeeb:Switch_ChocV1-hotswap, F.Cu at (296.5, 72.2)
- added SW42: Switch, zzkeeb:Switch_ChocV1-hotswap, F.Cu at (296.5, 90.3)
- added SW43: Switch, zzkeeb:Switch_ChocV1-hotswap, F.Cu at (296.5, 108.5)
- added SW44: Switch, zzkeeb:Switch_ChocV1-hotswap, F.Cu at (277.8, 132.7)
- added SW45: Switch, zzkeeb:Switch_ChocV1-hotswap, F.Cu at (315.0, 58.0)
- added SW46: Switch, zzkeeb:Switch_ChocV1-hotswap, F.Cu at (315.0, 75.5)
- added SW47: Switch, zzkeeb:Switch_ChocV1-hotswap, F.Cu at (315.0, 93.7)
- added SW48: Switch, zzkeeb:Switch_ChocV1-hotswap, F.Cu at (315.0, 111.8)
- added SW49: Switch, zzkeeb:Switch_ChocV1-hotswap, F.Cu at (295.5, 131.0)
- added SW5: Switch, zzkeeb:Switch_ChocV1-hotswap, F.Cu at (111.5, 70.0)
- added SW50: Switch, zzkeeb:Switch_ChocV1-hotswap, F.Cu at (336.0, 64.5)
- added SW51: Switch, zzkeeb:Switch_ChocV1-hotswap, F.Cu at (336.0, 82.7)
- added SW52: Switch, zzkeeb:Switch_ChocV1-hotswap, F.Cu at (336.0, 100.8)
- added SW53: Switch, zzkeeb:Switch_ChocV1-hotswap, F.Cu at (336.0, 119.0)
- added SW54: Switch, zzkeeb:Switch_ChocV1-hotswap, F.Cu at (314.0, 133.5)
- added SW55: Switch, zzkeeb:Switch_ChocV1-hotswap, F.Cu at (353.5, 65.0)
- added SW56: Switch, zzkeeb:Switch_ChocV1-hotswap, F.Cu at (353.5, 83.2)
- added SW57: Switch, zzkeeb:Switch_ChocV1-hotswap, F.Cu at (353.5, 101.3)
- added SW58: Switch, zzkeeb:Switch_ChocV1-hotswap, F.Cu at (353.5, 119.5)
- added SW6: Switch, zzkeeb:Switch_ChocV1-hotswap, F.Cu at (111.5, 87.0)
- added SW7: Switch, zzkeeb:Switch_ChocV1-hotswap, F.Cu at (111.5, 104.0)
- added SW8: Switch, zzkeeb:Switch_ChocV1-hotswap, F.Cu at (111.5, 121.0)
- added SW9: Switch, zzkeeb:Switch_ChocV1-hotswap, F.Cu at (129.5, 129.1)
- added U1: MCU_rp2040-zero, zzkeeb:MCU_rp2040-zero-smd, F.Cu at (219.0, 61.0)
Other:
- board outline added: 308.5 x 121 mm

Commit message: Both halves
Parts:
- moved SW54 21.0 mm to (302.7, 115.8)
- moved SW49 20.8 mm to (284.7, 113.3)
- moved SW44 20.2 mm to (266.7, 115.8)
- moved SW38 18.8 mm to (266.7, 98.8)
- moved SW53 18.4 mm to (320.7, 108.8)
- moved SW58 18.3 mm to (338.7, 108.8)
- moved SW39 18.0 mm to (245.7, 121.3), turned to 22 degrees
- moved SW48 17.9 mm to (302.7, 98.8)
- moved SW37 17.9 mm to (266.7, 81.8)
- moved SW52 17.8 mm to (320.7, 91.8)
- moved SW57 17.6 mm to (338.7, 91.8)
- moved SW51 17.2 mm to (320.7, 74.8)
- moved SW47 17.1 mm to (302.7, 81.8)
- moved SW56 17.0 mm to (338.7, 74.8)
- moved SW43 17.0 mm to (284.7, 96.3)
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Other:
- board outline removed

Commit message: First version
Parts:
- D1, D10, D11, D12, D13, D14, D15, D16, D17, D18, D19, D2, D20, D21, D22, D23, D24, D25, D26, D27, D28, D29, D3, D30, D31, D32, D33, D34, D35, D36, D37, D38, D39, D4, D40, D41, D42, D43, D44, D45, D46, D47, D48, D49, D5, D50, D51, D52, D53, D54, D55, D56, D57, D58, D6, D7, D8, D9: moved to B.Cu
- moved D58 316.5 mm to (336.9, 99.4), turned to -165 degrees
- moved D53 311.2 mm to (319.4, 104.1), turned to -165 degrees
- moved D57 306.8 mm to (332.4, 82.9), turned to -165 degrees
- moved D54 302.2 mm to (303.8, 115.4), turned to -165 degrees
- moved D52 300.9 mm to (315.1, 87.6), turned to -165 degrees
- moved D56 297.7 mm to (328.0, 66.5), turned to -165 degrees
- moved D51 290.9 mm to (310.7, 71.2), turned to -165 degrees
- moved D55 289.0 mm to (323.6, 50.1), turned to -165 degrees
- moved D48 287.9 mm to (299.6, 99.0), turned to -165 degrees
- moved D44 284.0 mm to (269.1, 124.8), turned to -165 degrees
- moved D49 283.9 mm to (286.0, 117.6), turned to -165 degrees
- moved D43 282.2 mm to (281.5, 101.3), turned to -165 degrees
- moved D47 277.9 mm to (295.1, 82.6), turned to -165 degrees
- moved D39 276.0 mm to (263.4, 128.6), turned to -165 degrees
- moved D50 273.9 mm to (306.4, 54.9), turned to -165 degrees
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Routing:
- net Net-(D35-A): track 0.00 -> 0.64 mm
Other:
- board outline added: 279.6 x 121.9 mm

Commit message: Improved shape in fusion360. Bit bigger and smooth curve.
Parts:
- moved D29 13.0 mm to (195.2, 144.8)
- moved D34 12.0 mm to (239.7, 144.8)
- moved D39 11.1 mm to (254.7, 135.5)
- moved D24 10.2 mm to (181.2, 135.6)
Routing:
- net col6: track 0.00 -> 89.0 mm
- net col10: track 0.00 -> 75.8 mm
- net col9: track 0.00 -> 56.3 mm
- net col11: track 0.00 -> 55.4 mm
- net col8: track 0.00 -> 55.3 mm
- net col7: track 0.00 -> 55.0 mm
- net Net-(D34-A): track 0.00 -> 17.5 mm
- net Net-(D39-A): track 0.00 -> 13.2 mm
- net Net-(D38-A): track 0.00 -> 11.3 mm
- net Net-(D31-A): track 0.00 -> 10.9 mm
- net Net-(D32-A): track 0.00 -> 10.9 mm
- net Net-(D45-A): track 0.00 -> 10.8 mm
- net Net-(D57-A): track 0.00 -> 10.8 mm
- net Net-(D56-A): track 0.00 -> 10.8 mm
- net Net-(D54-A): track 0.00 -> 10.8 mm
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Other:
- board size 279.6 x 121.9 mm -> 281.5 x 124.7 mm

Commit message: Place diodes differently
Parts:
- moved D34 10.9 mm to (234.3, 154.3), turned to -75 degrees
- moved D24 10.5 mm to (170.9, 133.8), turned to -105 degrees
- moved D39 8.52 mm to (249.3, 142.1), turned to -75 degrees
- moved D29 8.47 mm to (186.7, 145.4), turned to -105 degrees
- moved D18 5.49 mm to (139.8, 102.2), turned to -105 degrees
- moved D26 5.48 mm to (182.0, 83.5), turned to -105 degrees
- moved D8 5.43 mm to (101.8, 104.9), turned to -105 degrees
- moved D5 5.43 mm to (115.0, 55.7), turned to -105 degrees
- moved D17 5.42 mm to (144.2, 85.8), turned to -105 degrees
- moved D21 5.40 mm to (165.3, 76.4), turned to -105 degrees
- moved D23 5.40 mm to (156.5, 109.3), turned to -105 degrees
- moved D16 5.39 mm to (148.6, 69.3), turned to -105 degrees
- moved D20 5.39 mm to (169.7, 60.0), turned to -105 degrees
- moved D10 5.38 mm to (134.9, 50.7), turned to -105 degrees
- moved D19 5.37 mm to (152.1, 125.7), turned to -105 degrees
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Connections:
- U1 pad 15: col5 -> col0
- U1 pad 16: col4 -> col1
- U1 pad 17: col3 -> col2
- U1 pad 18: col2 -> col3
- U1 pad 19: col1 -> col4
- U1 pad 20: col0 -> col5
- U1 pad 4: col6 -> col11
- U1 pad 5: col7 -> col10
- U1 pad 6: col8 -> col9
- U1 pad 7: col9 -> col8
- U1 pad 8: col10 -> col7
- U1 pad 9: col11 -> col6
Routing:
- net col11: track 55.4 -> 184.2 mm, vias 0 -> 1
- net col10: track 75.8 -> 193.7 mm, vias 0 -> 1
- net row0: track 0.00 -> 38.5 mm
- net col6: track 89.0 -> 69.8 mm
- net Net-(D34-A): track 17.5 -> 0.00 mm
- net Net-(D39-A): track 13.2 -> 0.00 mm
- net Net-(D35-A): track 11.3 -> 0.00 mm
- net Net-(D38-A): track 11.3 -> 0.00 mm
- net Net-(D31-A): track 10.9 -> 0.00 mm
- net Net-(D32-A): track 10.9 -> 0.00 mm
- net Net-(D45-A): track 10.8 -> 0.00 mm
- net Net-(D57-A): track 10.8 -> 0.00 mm
- net Net-(D56-A): track 10.8 -> 0.00 mm
- net Net-(D54-A): track 10.8 -> 0.00 mm
- net Net-(D33-A): track 10.7 -> 0.00 mm
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
Commit message: Routing the right half WIP
Routing:
- net row3: track 0.00 -> 104.5 mm, vias 0 -> 6
- net row2: track 0.00 -> 104.3 mm, vias 0 -> 6
- net row0: track 38.5 -> 0.00 mm
- net col7: track 54.7 -> 85.4 mm
- net col8: track 55.3 -> 84.6 mm
- net col9: track 56.1 -> 84.0 mm
- net col6: track 69.8 -> 89.6 mm
- net Net-(D34-A): track 0.00 -> 7.69 mm
- net Net-(D45-A): track 0.00 -> 5.94 mm
- net Net-(D52-A): track 0.00 -> 5.72 mm
- net Net-(D46-A): track 0.00 -> 5.71 mm
- net Net-(D55-A): track 0.00 -> 5.70 mm
- net Net-(D39-A): track 0.00 -> 5.68 mm
- net Net-(D56-A): track 0.00 -> 5.66 mm
- net Net-(D57-A): track 0.00 -> 5.66 mm
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
Commit message: Right half routed
Routing:
- net row1: track 0.00 -> 107.4 mm, vias 0 -> 6
- net row0: track 0.00 -> 104.4 mm, vias 0 -> 6
- net col9: track 84.0 -> 178.5 mm, vias 0 -> 1
- net col8: track 84.6 -> 164.2 mm, vias 0 -> 1
- net col7: track 85.4 -> 130.3 mm, vias 0 -> 1
- net col6: track 89.6 -> 116.2 mm, vias 0 -> 1
- net row3: track 104.5 -> 106.3 mm

Commit message: Routing done
Parts:
- moved D9 5.41 mm to (117.3, 116.4), turned to -105 degrees
- moved D13 5.39 mm to (121.7, 99.9), turned to -105 degrees
- moved D12 5.34 mm to (126.1, 83.5), turned to -105 degrees
Connections:
- U1 pad 15: col0 -> col5
- U1 pad 16: col1 -> col4
- U1 pad 17: col2 -> col3
- U1 pad 18: col3 -> col2
- U1 pad 19: col4 -> col1
- U1 pad 20: col5 -> col0
Routing:
- net row4: track 0.00 -> 299.6 mm, vias 0 -> 11
- net row3: track 106.3 -> 319.5 mm, vias 6 -> 12
- net row0: track 104.4 -> 297.9 mm, vias 6 -> 14
- net col1: track 0.00 -> 190.4 mm, vias 0 -> 1
- net row2: track 104.3 -> 287.9 mm, vias 6 -> 14
- net col0: track 0.00 -> 179.6 mm, vias 0 -> 1
- net row1: track 107.4 -> 284.5 mm, vias 6 -> 14
- net col2: track 0.00 -> 169.4 mm, vias 0 -> 1
- net col3: track 0.00 -> 152.4 mm, vias 0 -> 1
- net col4: track 0.00 -> 121.6 mm, vias 0 -> 1
- net col5: track 0.00 -> 109.2 mm, vias 0 -> 1
- net Net-(D26-A): track 0.00 -> 4.30 mm
- net Net-(D21-A): track 0.00 -> 4.28 mm
- net Net-(D11-A): track 0.00 -> 4.28 mm
- net Net-(D16-A): track 0.00 -> 4.28 mm
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