File: SofleUnsplit.kicad_pcb (KiCad board)
At the start: 2 copper layers, 281.5 x 124.7 mm, 117 parts, among them SW1 Switch, SW10 Switch, SW11 Switch, SW12 Switch, SW13 Switch, SW14 Switch, SW15 Switch, SW16 Switch, SW17 Switch, SW18 Switch, SW19 Switch, SW2 Switch, SW20 Switch, SW21 Switch, SW22 Switch, SW23 Switch, SW24 Switch, SW25 Switch, SW26 Switch, SW27 Switch, SW28 Switch, SW29 Switch, SW3 Switch, SW30 Switch, SW31 Switch, SW32 Switch, SW33 Switch, SW34 Switch, SW35 Switch, SW36 Switch, SW37 Switch, SW38 Switch, SW39 Switch, SW4 Switch, SW40 Switch, SW41 Switch, SW42 Switch, SW43 Switch, SW44 Switch, SW45 Switch, SW46 Switch, SW47 Switch, SW48 Switch, SW49 Switch, SW5 Switch, SW50 Switch, SW51 Switch, SW52 Switch, SW53 Switch, SW54 Switch, SW55 Switch, SW56 Switch, SW57 Switch, SW58 Switch, SW6 Switch, SW7 Switch, SW8 Switch, SW9 Switch, U1 MCU_rp2040-zero

Commit message: Polishing, finishing
Parts:
- added J1: Conn_01x04, Connector_PinSocket_2.54mm:PinSocket_1x04_P2.54mm_Vertical, F.Cu at (213.9, 96.7)
- added Ref**: Val**, local:josef_adamcik_20mm_cu_mask, B.Cu at (218.6, 154.7)
- moved D24 0.13 mm to (171.1, 133.7)
- moved SW24 0.13 mm to (178.6, 140.3)
- moved D27 0.13 mm to (177.8, 99.8)
- moved D28 0.13 mm to (173.4, 116.3)
- moved SW27 0.13 mm to (185.3, 103.8)
- moved SW28 0.13 mm to (180.9, 120.3)
- moved D10 0.13 mm to (135.0, 50.6)
- moved D15 0.13 mm to (153.1, 52.8)
- moved SW10 0.13 mm to (142.5, 54.6)
- moved SW15 0.13 mm to (160.6, 56.8)
- moved D11 0.13 mm to (130.6, 67.0)
- moved D16 0.13 mm to (148.7, 69.3)
- moved D25 0.13 mm to (186.6, 67.0)
- moved D26 0.13 mm to (182.2, 83.4)
- moved D29 0.13 mm to (186.8, 145.3)
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Connections:
- U1 pad 1: unconnected-(U1-0-Pad1) -> SDA
- U1 pad 2: unconnected-(U1-1-Pad2) -> SCL
Routing:
- net GND: track 0.00 -> 46.0 mm, vias 0 -> 2
- net SCL: track 0.00 -> 43.1 mm, vias 0 -> 1
- net SDA: track 0.00 -> 42.1 mm, vias 0 -> 1
- net +5V: track 0.00 -> 41.4 mm, vias 0 -> 1
- net row0: track 297.9 -> 296.0 mm
- net row4: track 299.6 -> 298.1 mm
- net col6: track 116.2 -> 117.6 mm
Other:
- board text added: "GND"
- board text added: "PWR"
- board text added: "SCL"
- board text added: "SDA"
- board text added: "STÁŇA Choc v0.1"
- board text added: "https://adamcik.me"

Commit message: Finalising
Parts:
- removed Ref**: Val**, local:josef_adamcik_20mm_cu_mask
- J1: value Conn_01x04 -> Conn_01x05; footprint Connector_PinSocket_2.54mm:PinSocket_1x04_P2.54mm_Vertical -> Connector_PinSocket_2.54mm:PinSocket_1x05_P2.54mm_Vertical
- moved J1 1.17 mm to (213.3, 97.8)
Connections:
- J1 pad 1: +5V -> +3.3V
- J1 pad 2: SCL -> GP2
- J1 pad 3: SDA -> GP1
- J1 pad 4: GND -> GP0
- U1 pad 1: SDA -> GP0
- U1 pad 2: SCL -> GP1
- U1 pad 21: unconnected-(U1-3V3-Pad21) -> +3.3V
- U1 pad 23: +5V -> unconnected-(U1-5V-Pad23)
- U1 pad 3: unconnected-(U1-2-Pad3) -> GP2
Routing:
- net SCL: track 43.1 -> 0.00 mm, vias 1 -> 0
- net SDA: track 42.1 -> 0.00 mm, vias 1 -> 0
- net +5V: track 41.4 -> 0.00 mm, vias 1 -> 0
- net GP0: track 0.00 -> 39.6 mm, vias 0 -> 1
- net GP1: track 0.00 -> 38.5 mm, vias 0 -> 1
- net GP2: track 0.00 -> 38.1 mm, vias 0 -> 1
- net +3.3V: track 0.00 -> 32.9 mm, vias 0 -> 1
- net col1: track 190.4 -> 187.4 mm
- net GND: track 46.0 -> 49.0 mm, vias 2 -> 1
- net col2: track 169.4 -> 168.4 mm
- net col0: track 179.6 -> 178.7 mm
Other:
- board text added: "3.3V"
- board text added: "GP0"
- board text added: "GP1"
- board text added: "GP2"
- board text removed: "PWR"
- board text removed: "SCL"
- board text removed: "SDA"

Commit message: First version, final, before last check.
Parts:
- added G1: ~, local:josef_adamcik_20mm_cu_mask, B.Cu at (218.1, 154.6)
- added H1: MountingHole, MountingHole:MountingHole_2.7mm_M2.5_DIN965, F.Cu at (119.8, 47.0)
- added H2: MountingHole, MountingHole:MountingHole_2.7mm_M2.5_DIN965, F.Cu at (315.8, 47.0)
- added H3: MountingHole, MountingHole:MountingHole_2.7mm_M2.5_DIN965, F.Cu at (109.8, 122.0)
- added H4: MountingHole, MountingHole:MountingHole_2.7mm_M2.5_DIN965, F.Cu at (325.8, 122.0)
- added H5: MountingHole, MountingHole:MountingHole_3.2mm_M3_DIN965, F.Cu at (202.8, 99.0)
- added H6: MountingHole, MountingHole:MountingHole_3.2mm_M3_DIN965, F.Cu at (232.8, 99.0)
- added H7: MountingHole, MountingHole:MountingHole_3.2mm_M3_DIN965, F.Cu at (203.8, 147.0)
- added H8: MountingHole, MountingHole:MountingHole_3.2mm_M3_DIN965, F.Cu at (231.8, 147.0)
Routing:
- net GND: track 49.0 -> 0.71 mm, vias 1 -> 0
- net col10: track 191.4 -> 187.7 mm
- net col1: track 187.4 -> 185.3 mm
- added copper zone on B.Cu, net GND
- added copper zone on F.Cu, net GND

Commit message: Add placement for JLCPCB number
Other:
- board text added: "JLCJLCJLCJLC"
Changed lines of the file:
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@@
+    (effects (font (size 1 1) (thickness 0.15)) (justify left bottom mirror))
+  )
+  (gr_text "JLCJLCJLCJLC" (at 112.78 44.92) (layer "B.SilkS")
     (effects (font (size 1 1) (thickness 0.15)) (justify left bottom mirror))
   )

Commit message: Minor fixes
Routing:
- net GND: vias 0 -> 6
